File: saikoutype_nkbm-st110r2/pcb/NKBM-ST110r2.kicad_pcb (KiCad board)
At the start: 2 copper layers, 428.4 x 124.9 mm, 276 parts, among them K00 CHRY_MX, K02 CHRY_MX, K03 CHRY_MX, K04 CHRY_MX, K05 CHRY_MX, K06 CHRY_MX, K07 CHRY_MX, K08 CHRY_MX, K09 CHRY_MX, K0B CHRY_MX, K0C CHRY_MX, K0D CHRY_MX, K0E CHRY_MX, K10 CHRY_MX, K11 CHRY_MX, K12 CHRY_MX, K13 CHRY_MX, K14 CHRY_MX, K15 CHRY_MX, K16 CHRY_MX, K17 CHRY_MX, K18 CHRY_MX, K19 CHRY_MX, K1A CHRY_MX, K1B CHRY_MX, K1C CHRY_MX, K1D CHRY_MX, K1E CHRY_MX, K1E2 CHRY_MX, K20 CHRY_MX, K21 CHRY_MX, K22 CHRY_MX, K23 CHRY_MX, K24 CHRY_MX, K25 CHRY_MX, K26 CHRY_MX, K27 CHRY_MX, K28 CHRY_MX, K29 CHRY_MX, K2A CHRY_MX, K2B CHRY_MX, K2C CHRY_MX, K30 CHRY_MX, K31 CHRY_MX, K32 CHRY_MX, K33 CHRY_MX, K34 CHRY_MX, K35 CHRY_MX, K36 CHRY_MX, K37 CHRY_MX, K38 CHRY_MX, K39 CHRY_MX, K3A CHRY_MX, K3B CHRY_MX, K3C CHRY_MX, K3E CHRY_MX, K3E2 CHRY_MX, K40 CHRY_MX, K402 CHRY_MX, K41 CHRY_MX, K42 CHRY_MX, K43 CHRY_MX, K44 CHRY_MX, K45 CHRY_MX, K46 CHRY_MX, K47 CHRY_MX, K48 CHRY_MX, K49 CHRY_MX, K4A CHRY_MX, K4B CHRY_MX, K4C CHRY_MX, K4D CHRY_MX, K4D2 CHRY_MX, K50 CHRY_MX, K51 CHRY_MX, K511 CHRY_MX, K52 CHRY_MX, K521 CHRY_MX, K53 CHRY_MX, K54 CHRY_MX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

Commit message: Begin conversion to 最悪ゴミ
Parts:
- removed MCU1: Teesny++ 2.0, null_keyboard:TEENSY2.0++
- added REF**: VQFN-64-1EP_9x9mm_P0.5mm_EP5.4x5.4mm, dfn_qfn:VQFN-64-1EP_9x9mm_P0.5mm_EP5.4x5.4mm, F.Cu at (466.8, 63.5)
- added REF**: QFN-64-1EP_9x9mm_P0.5mm_EP5.4x5.4mm, dfn_qfn:QFN-64-1EP_9x9mm_P0.5mm_EP5.4x5.4mm, F.Cu at (424.9, 66.6)
Routing:
- net /COL_06: track 628.0 -> 542.0 mm
- net /ROW_03: track 464.9 -> 386.7 mm
- net /COL_14: track 595.5 -> 517.8 mm
- net /COL_04: track 619.6 -> 543.7 mm
- net /COL_03: track 582.5 -> 506.7 mm
- net /COL_07: track 701.5 -> 626.6 mm
- net /COL_05: track 645.8 -> 571.0 mm
- net /ROW_02: track 436.0 -> 361.7 mm
- net /ROW_06: track 471.5 -> 400.2 mm
- net /ROW_01: track 431.2 -> 364.4 mm
- net /ROW_00: track 525.4 -> 459.2 mm
- net /COL_01: track 621.7 -> 559.5 mm
- net /COL_00: track 628.9 -> 566.9 mm
- net /ROW_05: track 496.1 -> 437.8 mm
- net /ROW_04: track 478.0 -> 422.2 mm
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